Commit message: feat: Gazebo simülasyonunu tamamla ve hataları ayıkla

File: src/my_robot_description/urdf/my_robot.urdf.xacro (robot description, xacro)
@@ -7,16 +7,10 @@
       <visual>
         <origin xyz="0 0 0.05" rpy="0 0 0"/>
-        <geometry>
-          <box size="0.4 0.3 0.1"/>
-        </geometry>
-        <material name="blue">
-          <color rgba="0.0 0.0 0.8 1.0"/>
-        </material>
+        <geometry><box size="0.4 0.3 0.1"/></geometry>
+        <material name="blue"><color rgba="0.0 0.0 0.8 1.0"/></material>
       </visual>
       <collision>
         <origin xyz="0 0 0.05" rpy="0 0 0"/>
-        <geometry>
-          <box size="0.4 0.3 0.1"/>
-        </geometry>
+        <geometry><box size="0.4 0.3 0.1"/></geometry>
       </collision>
       <inertial>
@@ -29,16 +23,10 @@
             <visual>
                 <origin xyz="0 0 0" rpy="${pi/2} 0 0" />
-                <geometry>
-                    <cylinder radius="${wheel_radius}" length="${wheel_length}" />
-                </geometry>
-                <material name="grey">
-                    <color rgba="0.5 0.5 0.5 1.0" />
-                </material>
+                <geometry><cylinder radius="${wheel_radius}" length="${wheel_length}" /></geometry>
+                <material name="grey"><color rgba="0.5 0.5 0.5 1.0" /></material>
             </visual>
             <collision>
                 <origin xyz="0 0 0" rpy="${pi/2} 0 0" />
-                <geometry>
-                    <cylinder radius="${wheel_radius}" length="${wheel_length}" />
-                </geometry>
+                <geometry><cylinder radius="${wheel_radius}" length="${wheel_length}" /></geometry>
             </collision>
             <inertial>
@@ -46,5 +34,5 @@
                 <inertia ixx="0.001" ixy="0.0" ixz="0.0" iyy="0.001" iyz="0.0" izz="0.001"/>
             </inertial>
-         </link>
+        </link>
         <joint name="${prefix}_wheel_joint" type="continuous">
             <parent link="base_link"/>
@@ -57,46 +45,26 @@
     <xacro:wheel_macro prefix="left" reflect="-1" />
     <link name="caster_wheel_front_link">
-        <visual>
-            <geometry>
-                <sphere radius="0.03"/>
-            </geometry>
-            <material name="grey"/>
-        </visual>
-        <collision>
-            <geometry>
-                <sphere radius="0.03"/>
-            </geometry>
-        </collision>
-        <inertial>
-            <mass value="0.05"/>
-            <inertia ixx="0.0001" ixy="0.0" ixz="0.0" iyy="0.0001" iyz="0.0" izz="0.0001"/>
-        </inertial>
+    <visual><geometry><sphere radius="0.05"/></geometry><material name="grey"/></visual>
+    <collision><geometry><sphere radius="0.05"/></geometry></collision>
+    <inertial><mass value="0.05"/><inertia ixx="0.0001" ixy="0.0" ixz="0.0" iyy="0.0001" iyz="0.0" izz="0.0001"/></inertial>
     </link>
-    <joint name="caster_wheel_front_joint" type="fixed">
-        <parent link="base_link"/>
-        <child link="caster_wheel_front_link"/>
-        <origin xyz="-0.15 0 0"/>
-    </joint>
-    <link name="caster_wheel_back_link">
-        <visual>
-            <geometry>
-                <sphere radius="0.03"/>
-            </geometry>
-            <material name="grey"/>
-        </visual>
-        <collision>
-            <geometry>
-                <sphere radius="0.03"/>
-            </geometry>
-        </collision>
-        <inertial>
-            <mass value="0.05"/>
-            <inertia ixx="0.0001" ixy="0.0" ixz="0.0" iyy="0.0001" iyz="0.0" izz="0.0001"/>
-        </inertial>
-    </link>
-    <joint name="caster_wheel_back_joint" type="fixed">
-        <parent link="base_link"/>
-        <child link="caster_wheel_back_link"/>
-        <origin xyz="0.15 0 0"/>
-    </joint>
+    <joint name="caster_wheel_front_joint" type="fixed"><parent link="base_link"/><child link="caster_wheel_front_link"/><origin xyz="-0.15 0 0"/></joint>
+    <link name="caster_wheel_back_link"><visual><geometry><sphere radius="0.05"/></geometry><material name="grey"/></visual><collision><geometry><sphere radius="0.05"/></geometry></collision><inertial><mass value="0.05"/><inertia ixx="0.0001" ixy="0.0" ixz="0.0" iyy="0.0001" iyz="0.0" izz="0.0001"/></inertial></link>
+    <joint name="caster_wheel_back_joint" type="fixed"><parent link="base_link"/><child link="caster_wheel_back_link"/><origin xyz="0.15 0 0"/></joint>
+    <gazebo>
+        <plugin filename="gz-sim-diff-drive-system" name="gz::sim::systems::DiffDrive">
+            <left_joint>left_wheel_joint</left_joint>
+            <right_joint>right_wheel_joint</right_joint>
+            <wheel_separation>-0.34</wheel_separation>
+            <wheel_radius>${wheel_radius}</wheel_radius>
+            <topic>/cmd_vel</topic>
+            <odom_topic>/odom</odom_topic>
+            <tf_topic>/tf</tf_topic>
+            <frame_id>odom</frame_id>
+            <child_frame_id>base_link</child_frame_id>
+        </plugin>
+        <plugin filename="gz-sim-joint-state-publisher-system" name="gz::sim::systems::JointStatePublisher">
+            <topic>/joint_states</topic>
+        </plugin>
+    </gazebo>
 </robot>

Commit message: fix: Tekerleklere sürtünme eklenerek odometri kayması düzeltildi

File: src/my_robot_description/urdf/my_robot.urdf.xacro (robot description, xacro)
@@ -26,8 +26,18 @@
                 <material name="grey"><color rgba="0.5 0.5 0.5 1.0" /></material>
             </visual>
-            <collision>
-                <origin xyz="0 0 0" rpy="${pi/2} 0 0" />
-                <geometry><cylinder radius="${wheel_radius}" length="${wheel_length}" /></geometry>
-            </collision>
+           <collision>
+            <origin xyz="0 0 0" rpy="${pi/2} 0 0" />
+            <geometry>
+                <cylinder radius="${wheel_radius}" length="${wheel_length}" />
+            </geometry>
+            <surface>
+              <friction>
+                <ode>
+                  <mu>1.0</mu>
+                  <mu2>1.0</mu2>
+                </ode>
+              </friction>
+            </surface>
+        </collision>
             <inertial>
                 <mass value="${wheel_mass}"/>

Commit message: chore: Formatlama ve satır sonu karakterlerini düzelt

File: src/my_robot_description/urdf/my_robot.urdf.xacro (robot description, xacro)
@@ -55,7 +55,7 @@
     <xacro:wheel_macro prefix="left" reflect="-1" />
     <link name="caster_wheel_front_link">
-    <visual><geometry><sphere radius="0.05"/></geometry><material name="grey"/></visual>
-    <collision><geometry><sphere radius="0.05"/></geometry></collision>
-    <inertial><mass value="0.05"/><inertia ixx="0.0001" ixy="0.0" ixz="0.0" iyy="0.0001" iyz="0.0" izz="0.0001"/></inertial>
+     <visual><geometry><sphere radius="0.05"/></geometry><material name="grey"/></visual>
+     <collision><geometry><sphere radius="0.05"/></geometry></collision>
+     <inertial><mass value="0.05"/><inertia ixx="0.0001" ixy="0.0" ixz="0.0" iyy="0.0001" iyz="0.0" izz="0.0001"/></inertial>
     </link>
     <joint name="caster_wheel_front_joint" type="fixed"><parent link="base_link"/><child link="caster_wheel_front_link"/><origin xyz="-0.15 0 0"/></joint>
